File: Rev. 0/Eagle/PET_1541_Ada.sch (EAGLE design)
At the start: 33 parts, among them IC1 74LS06N, IC2 74LS04N, J1 PET-USERPORT, J3 010599, J4 FCR681465P, SW6 JPT1236HB

Commit message: CB2 Silk screen fix
Connections:
- net CA2 renamed CB2
Changed lines of the file:
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@@
 </segment>
 </net>
-<net name="CA2" class="0">
+<net name="CB2" class="0">
 <segment>
 <pinref part="J1" gate="G$1" pin="CB2"/>
